Commit message: 新增 myrobot_gazebo 包 + 模型支持 Gazebo（惯性参数/可切换硬件插件）
- myrobot_gazebo: 仿真世界(桌子+目标方块) + gazebo.launch.xml + 控制器配置
- 模型 URDF: 补 11 个 link 的惯性参数，ros2_control 宏支持 sim_mode 切换
  mock_components/GenericSystem ↔ gazebo_ros2_control/GazeboSystem
- 注: 当前环境 gazebo_ros2_control 0.4.10 与 ros2_control 2.54 插件基类不兼容，
  Gazebo 运行需待环境升级，mock 链路不受影响

File: src/myrobot_description/urdf/arm.xacro (robot description, xacro)
@@ -18,4 +18,9 @@
             <origin xyz="0 0 0.05" rpy="0.0 0.0 0.0"/>
         </collision>
+        <inertial>
+            <mass value="5.0"/>
+            <origin xyz="0 0 0.05" rpy="0 0 0"/>
+            <inertia ixx="0.0708" ixy="0.0" ixz="0.0" iyy="0.0708" iyz="0.0" izz="0.1333"/>
+        </inertial>
     </link>
     <!-- 第一个轴 -->
@@ -34,4 +39,9 @@
             <origin xyz = "0 0 0.25" rpy="0 0 0"/>
         </collision>
+        <inertial>
+            <mass value="2.0"/>
+            <origin xyz="0 0 0.25" rpy="0 0 0"/>
+            <inertia ixx="0.0483" ixy="0.0" ixz="0.0" iyy="0.0483" iyz="0.0" izz="0.0133"/>
+        </inertial>
     </link>
     <!-- 第2个轴 -->
@@ -50,4 +60,9 @@
             <origin xyz = "0 0 0.3" rpy="0 0 0"/>
         </collision>
+        <inertial>
+            <mass value="1.0"/>
+            <origin xyz="0 0 0.3" rpy="0 0 0"/>
+            <inertia ixx="0.0308" ixy="0.0" ixz="0.0" iyy="0.0308" iyz="0.0" izz="0.0017"/>
+        </inertial>
     </link>
     <!-- 第3个轴 -->
@@ -66,4 +81,9 @@
             <origin xyz = "0 0 0.05" rpy="0 0 0"/>
         </collision>
+        <inertial>
+            <mass value="0.5"/>
+            <origin xyz="0 0 0.05" rpy="0 0 0"/>
+            <inertia ixx="0.0008" ixy="0.0" ixz="0.0" iyy="0.0008" iyz="0.0" izz="0.0008"/>
+        </inertial>
     </link>
     <!-- 第4个轴 -->
@@ -82,4 +102,9 @@
             <origin xyz = "0 0 0.25" rpy="0 0 0"/>
         </collision>
+        <inertial>
+            <mass value="0.8"/>
+            <origin xyz="0 0 0.25" rpy="0 0 0"/>
+            <inertia ixx="0.0173" ixy="0.0" ixz="0.0" iyy="0.0173" iyz="0.0" izz="0.0013"/>
+        </inertial>
     </link>
     <!-- 第5个轴 -->
@@ -99,4 +124,9 @@
             <origin xyz = "0 0 0.025" rpy="0 0 0"/>
         </collision>
+        <inertial>
+            <mass value="0.3"/>
+            <origin xyz="0 0 0.025" rpy="0 0 0"/>
+            <inertia ixx="0.0003" ixy="0.0" ixz="0.0" iyy="0.0003" iyz="0.0" izz="0.0005"/>
+        </inertial>
     </link>
     <!-- 第6个轴 -->
@@ -116,7 +146,17 @@
             <origin xyz = "0 0 0.01" rpy="0 0 0"/>
         </collision>
+        <inertial>
+            <mass value="0.2"/>
+            <origin xyz="0 0 0.01" rpy="0 0 0"/>
+            <inertia ixx="0.0002" ixy="0.0" ixz="0.0" iyy="0.0002" iyz="0.0" izz="0.0003"/>
+        </inertial>
     </link>
     <!-- 模拟夹抓工具 -->
     <link name="tool_link">
+        <inertial>
+            <mass value="0.01"/>
+            <origin xyz="0 0 0" rpy="0 0 0"/>
+            <inertia ixx="0.0000002" ixy="0.0" ixz="0.0" iyy="0.0000002" iyz="0.0" izz="0.0000002"/>
+        </inertial>
     </link>
     <joint name="joint1" type="revolute">    <!--可旋转-->
@@ -167,4 +207,2 @@
     </joint>
 </robot>
-<!-- sudo apt install ros-humble-urdf-tutorial -->
-<!-- ros2 launch urdf_tutorial display.launch.py model:=/home/zhz/robot_arm_ws/src/myrobot_description/urdf/arm.urdf -->

File: src/myrobot_description/urdf/gripper.xacro (robot description, xacro)
@@ -15,4 +15,9 @@
             <origin xyz="0.0 0.0 0.01" rpy="0.0 0.0 0.0"/>
         </collision>
+        <inertial>
+            <mass value="0.3"/>
+            <origin xyz="0 0 0.01" rpy="0 0 0"/>
+            <inertia ixx="0.0001" ixy="0.0" ixz="0.0" iyy="0.0010" iyz="0.0" izz="0.0011"/>
+        </inertial>
     </link>
     <link name="gripper_left_finger_link">
@@ -30,4 +35,9 @@
             <origin xyz="0.0 0.0 0.04" rpy="0.0 0.0 0.0"/>
         </collision>
+        <inertial>
+            <mass value="0.1"/>
+            <origin xyz="0 0 0.04" rpy="0 0 0"/>
+            <inertia ixx="0.00008" ixy="0.0" ixz="0.0" iyy="0.00006" iyz="0.0" izz="0.00003"/>
+        </inertial>
     </link>
     <link name="gripper_right_finger_link">
@@ -45,4 +55,9 @@
             <origin xyz="0.0 0.0 0.04" rpy="0.0 0.0 0.0"/>
         </collision>
+        <inertial>
+            <mass value="0.1"/>
+            <origin xyz="0 0 0.04" rpy="0 0 0"/>
+            <inertia ixx="0.00008" ixy="0.0" ixz="0.0" iyy="0.00006" iyz="0.0" izz="0.00003"/>
+        </inertial>
     </link>
     <joint name="gripper_left_finger_joint" type="prismatic">

File: src/myrobot_description/urdf/my_robot.ros2_control.xacro (robot description, xacro)
@@ -4,11 +4,17 @@
         统一的 ros2_control 硬件块（宏版，单一来源）。
         关节初始位置由 urdf/initial_positions.yaml 驱动，改初值不需要动 xacro。
+        sim_mode: mock=虚拟硬件 | gazebo=物理仿真（gazebo_ros2_control）
     -->
-    <xacro:macro name="my_robot_ros2_control" params="name initial_positions_file">
+    <xacro:macro name="my_robot_ros2_control"
+                 params="name initial_positions_file sim_mode:=mock">
         <xacro:property name="initial_positions" value="${xacro.load_yaml(initial_positions_file)['initial_positions']}"/>
         <ros2_control name="${name}" type="system">
             <hardware>
-                <!-- By default, set up controllers for simulation. This won't work on real hardware -->
-                <plugin>mock_components/GenericSystem</plugin>
+                <xacro:if value="${sim_mode == 'gazebo'}">
+                    <plugin>gazebo_ros2_control/GazeboSystem</plugin>
+                </xacro:if>
+                <xacro:unless value="${sim_mode == 'gazebo'}">
+                    <plugin>mock_components/GenericSystem</plugin>
+                </xacro:unless>
             </hardware>
             <joint name="joint1">

File: src/myrobot_description/urdf/myrobot_urdf.xacro (robot description, xacro)
@@ -1,4 +1,6 @@
 <?xml version="1.0"?>
 <robot name="my_robot" xmlns:xacro="http://www.ros.org/wiki/xacro">
+    <!-- sim_mode: mock=虚拟硬件(默认) | gazebo=物理仿真 -->
+    <xacro:arg name="sim_mode" default="mock"/>
     <xacro:include filename="common_properties.xacro"/>
     <xacro:include filename="arm.xacro"/>
@@ -7,5 +9,6 @@
     <!-- 生成 ros2_control 硬件块，初始位置从 initial_positions.yaml 读取 -->
     <xacro:my_robot_ros2_control name="Arm"
-         initial_positions_file="$(find myrobot_description)/urdf/initial_positions.yaml"/>
+         initial_positions_file="$(find myrobot_description)/urdf/initial_positions.yaml"
+         sim_mode="$(arg sim_mode)"/>
     <joint name="gripper_base_joint" type="fixed">
         <parent link="tool_link"/>
