Commit message: Gazebo 集成补丁 + 进度文档
- gazebo_ros2_control 0.4.10 源码补丁适配 ros2_control 2.54：
  插件注册基类改为 SystemInterface（XML + 源码宏 + 索引导出）
- URDF 增加 gazebo 插件块（sim_mode=gazebo 时生成）
- gazebo.launch.xml 修正架构（无需外部 ros2_control_node）
- 新增 进度.md 项目进度总结
- 清理测试残留文件

File: src/myrobot_description/urdf/myrobot_urdf.xacro (robot description, xacro)
@@ -11,4 +11,13 @@
          initial_positions_file="$(find myrobot_description)/urdf/initial_positions.yaml"
          sim_mode="$(arg sim_mode)"/>
+    <!-- Gazebo 模式：加载控制插件（gzserver 内部自建 controller_manager） -->
+    <xacro:property name="sim_mode_value" value="$(arg sim_mode)"/>
+    <xacro:if value="${sim_mode_value == 'gazebo'}">
+        <gazebo>
+            <plugin name="gazebo_ros2_control" filename="libgazebo_ros2_control.so">
+                <parameters>$(find myrobot_gazebo)/config/ros2_controllers.yaml</parameters>
+            </plugin>
+        </gazebo>
+    </xacro:if>
     <joint name="gripper_base_joint" type="fixed">
         <parent link="tool_link"/>
