Commit message: Gazebo 端到端跑通：世界离线化 + 插件注册修复 + use_sim_time 对齐 + 物理抓取优化
- world: model://ground_plane/sun 改内联，避免 gzserver 卡在线模型数据库
- gazebo_ros2_control: 注册基类改回 GazeboSystemInterface（gzserver 插件加载）；
  控制方式改 per-joint（is_pos_pid），避免无增益关节力控瘫软
- use_sim_time: move_group.launch.py 重写支持参数；gazebo launch 全节点对齐仿真时钟
- 物理抓取: 手指碰撞 0.2→0.02；夹爪 position_pid 力控；双指显式控制
  （Gazebo 不执行 URDF mimic）；高摩擦 mu=5；笛卡尔路径 + 抓取高度 0.51
  （补偿固定关节 lumping 丢失的 2cm 偏移）
- grasp_demo: 支持 world=mock|gazebo 参数（gazebo 坐标+笛卡尔）
- 对接文档/进度文档更新（含遗留问题与证据日志）

File: src/myrobot_description/urdf/gripper.xacro (robot description, xacro)
@@ -31,5 +31,5 @@
         <collision>
             <geometry>
-                <box size="0.2 0.06 0.08"/>
+                <box size="0.02 0.06 0.08"/>
             </geometry>
             <origin xyz="0.0 0.0 0.04" rpy="0.0 0.0 0.0"/>
@@ -51,5 +51,5 @@
         <collision>
             <geometry>
-                <box size="0.2 0.06 0.08"/>
+                <box size="0.02 0.06 0.08"/>
             </geometry>
             <origin xyz="0.0 0.0 0.04" rpy="0.0 0.0 0.0"/>
@@ -73,5 +73,7 @@
         <origin xyz="0.07 0.0 0.02" rpy="0.0 0.0 0.0"/>
         <axis xyz="1 0.0 0.0"/>
-        <mimic joint="gripper_left_finger_joint" multiplier="-1.0"/>
+        <!-- 注意：不用 <mimic>！Gazebo 11 不执行 URDF mimic（右指会变成自由关节），
+             且 MoveIt 不会把 mimic 关节写入控制轨迹。右指由 ros2_control 显式控制，
+             目标值 = -左指（见 SRDF group_state 与 grasp_demo） -->
         <limit lower="-0.06" upper="0.0" effort="1000.0" velocity="1.0"/>
     </joint>

File: src/myrobot_description/urdf/my_robot.ros2_control.xacro (robot description, xacro)
@@ -55,7 +55,33 @@
             </joint>
             <joint name="gripper_left_finger_joint">
-                <command_interface name="position"/>
+                <!-- gazebo：力控（POSITION_PID，SetForce 夹持），避免 SetPosition
+                     瞬移把抓取物体挤飞；mock：普通 position 接口 -->
+                <xacro:if value="${sim_mode == 'gazebo'}">
+                    <command_interface name="position_pid"/>
+                    <param name="pos_kp">500.0</param>
+                    <param name="pos_ki">0.0</param>
+                    <param name="pos_kd">15.0</param>
+                </xacro:if>
+                <xacro:unless value="${sim_mode == 'gazebo'}">
+                    <command_interface name="position"/>
+                </xacro:unless>
                 <state_interface name="position">
                   <param name="initial_value">${initial_positions['gripper_left_finger_joint']}</param>
+                </state_interface>
+            </joint>
+            <!-- 右手指：Gazebo 不执行 URDF 的 <mimic>，必须显式纳入 ros2_control
+                 由控制器按 -left 目标驱动（MoveIt 会经 mimic 推导右指目标值） -->
+            <joint name="gripper_right_finger_joint">
+                <xacro:if value="${sim_mode == 'gazebo'}">
+                    <command_interface name="position_pid"/>
+                    <param name="pos_kp">500.0</param>
+                    <param name="pos_ki">0.0</param>
+                    <param name="pos_kd">15.0</param>
+                </xacro:if>
+                <xacro:unless value="${sim_mode == 'gazebo'}">
+                    <command_interface name="position"/>
+                </xacro:unless>
+                <state_interface name="position">
+                  <param name="initial_value">${initial_positions['gripper_right_finger_joint']}</param>
                 </state_interface>
             </joint>

File: src/myrobot_description/urdf/myrobot_urdf.xacro (robot description, xacro)
@@ -25,3 +25,13 @@
         <origin xyz="0.0 0.0 0.0" rpy="0.0 0.0 0.0"/>
     </joint>
+    <!-- 手指高摩擦（mu=5）：Gazebo 默认 mu=1 偏低，夹爪力控夹持时方块容易
+         从指间滑脱；提高摩擦后夹持更可靠（配合 POSITION_PID 力控夹爪） -->
+    <gazebo reference="gripper_left_finger_link">
+        <mu1>5.0</mu1>
+        <mu2>5.0</mu2>
+    </gazebo>
+    <gazebo reference="gripper_right_finger_link">
+        <mu1>5.0</mu1>
+        <mu2>5.0</mu2>
+    </gazebo>
 </robot>

Commit message: Gazebo 物理抓取稳定化 + 项目文档整理
- 新增抓取附着插件 myrobot_grasp_attach（/gazebo_grasp_attach 服务）：
  到位后把目标方块附着到 hand_link，配合 gripper_grasp_5cm 轻夹（±0.0355）
  与夹爪 effort 限位 2.0，消除接触瞬态把方块弹飞的问题
- grasp_demo：Planning Scene 同步桌面/方块避障；确定性 PTP 关节中间位
  代替 OMPL 随机路径；低速带载（0.08/0.04）；gazebo 模式完整流程
- 世界：桌子 static 防漂移；方块挂载附着插件
- URDF：base_link kinematic 锚定（防整机漂移与 TF 分离）；夹爪 effort 限位
- 文档：README 重写为项目级说明；新增使用手册.md；删除智能体交接文档
  （对接文档.md、进度.md）

File: src/myrobot_description/urdf/gripper.xacro (robot description, xacro)
@@ -66,5 +66,5 @@
         <origin xyz="-0.07 0.0 0.02" rpy="0.0 0.0 0.0"/>
         <axis xyz="1 0.0 0.0"/>
-        <limit lower="0.0" upper="0.06" effort="1000.0" velocity="1.0"/>
+        <limit lower="0.0" upper="0.06" effort="2.0" velocity="1.0"/>
     </joint>
     <joint name="gripper_right_finger_joint" type="prismatic">
@@ -76,5 +76,5 @@
              且 MoveIt 不会把 mimic 关节写入控制轨迹。右指由 ros2_control 显式控制，
              目标值 = -左指（见 SRDF group_state 与 grasp_demo） -->
-        <limit lower="-0.06" upper="0.0" effort="1000.0" velocity="1.0"/>
+        <limit lower="-0.06" upper="0.0" effort="2.0" velocity="1.0"/>
     </joint>
 </robot>

File: src/myrobot_description/urdf/my_robot.ros2_control.xacro (robot description, xacro)
@@ -58,8 +58,5 @@
                      瞬移把抓取物体挤飞；mock：普通 position 接口 -->
                 <xacro:if value="${sim_mode == 'gazebo'}">
-                    <command_interface name="position_pid"/>
-                    <param name="pos_kp">500.0</param>
-                    <param name="pos_ki">0.0</param>
-                    <param name="pos_kd">15.0</param>
+                    <command_interface name="position"/>
                 </xacro:if>
                 <xacro:unless value="${sim_mode == 'gazebo'}">
@@ -74,8 +71,5 @@
             <joint name="gripper_right_finger_joint">
                 <xacro:if value="${sim_mode == 'gazebo'}">
-                    <command_interface name="position_pid"/>
-                    <param name="pos_kp">500.0</param>
-                    <param name="pos_ki">0.0</param>
-                    <param name="pos_kd">15.0</param>
+                    <command_interface name="position"/>
                 </xacro:if>
                 <xacro:unless value="${sim_mode == 'gazebo'}">

File: src/myrobot_description/urdf/myrobot_urdf.xacro (robot description, xacro)
@@ -14,4 +14,9 @@
     <xacro:property name="sim_mode_value" value="$(arg sim_mode)"/>
     <xacro:if value="${sim_mode_value == 'gazebo'}">
+        <!-- 锚定根链接；否则整个机械臂会在重力/关节反力下漂移，而 TF 仍把
+             base_link 当作固定世界坐标，导致规划位姿与 Gazebo 物理位姿分离。 -->
+        <gazebo reference="base_link">
+            <kinematic>true</kinematic>
+        </gazebo>
         <gazebo>
             <plugin name="gazebo_ros2_control" filename="libgazebo_ros2_control.so">
